Commit message: feat: add R550 large Ackermann meshes from vehicle

File: r550_description/urdf/r550_ackermann.urdf (robot description, URDF)
Before this commit: robot r550_ackermann, 12 links, 11 joints
Links:
- link base_link: geometry collision box size=0.762 0.35 0.15; visual mesh filename=package://r550_description/meshes/r550_ackermann/base_link.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
- link camera_link: geometry collision box size=0.04 0.08 0.04; visual mesh filename=package://r550_description/meshes/r550_ackermann/camera.STL
- link front_left_wheel_link: geometry collision cylinder length=0.08 radius=0.12; visual mesh filename=package://r550_description/meshes/r550_ackermann/front_left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
- link front_right_wheel_link: geometry collision cylinder length=0.08 radius=0.12; visual mesh filename=package://r550_description/meshes/r550_ackermann/front_righ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
- link laser: geometry collision cylinder length=0.05 radius=0.03; visual mesh filename=package://r550_description/meshes/r550_ackermann/laser.STL
- link rear_left_wheel_link: geometry collision cylinder length=0.08 radius=0.12; visual mesh filename=package://r550_description/meshes/r550_ackermann/rear_left_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
- link rear_right_wheel_link: geometry collision cylinder length=0.08 radius=0.12; visual mesh filename=package://r550_description/meshes/r550_ackermann/rear_right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

Commit message: fix: align R550 mesh model with vehicle kinematics

File: r550_description/urdf/r550_ackermann.urdf (robot description, URDF)
Before this commit: robot r550_ackermann, 12 links, 11 joints
Links:
- link base_link: geometry collision box size=0.76 0.60 0.20; visual mesh filename=package://r550_description/meshes/r550_ackermann/base_link.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
Joints:
- joint base_footprint_joint: origin xyz=0 0 0.12 rpy=0 0 0 -> xyz=0 0 0 rpy=0 0 0
- joint camera_joint: origin xyz=0.58 0 0.32 rpy=0 0 0 -> xyz=0.3204 -0.0016 0.1321 rpy=0 0 0
- joint front_left_steer_joint: origin xyz=0.53 0.295 0.12 rpy=0 0 0 -> xyz=0.2808 0.2188 0.01149 rpy=0 0 0
- joint front_left_wheel_joint: origin xyz=0 0 0 rpy=0 0 0 -> xyz=-0.000739 0.0743 -0.0373 rpy=0 0 0
- joint front_right_steer_joint: origin xyz=0.53 -0.295 0.12 rpy=0 0 0 -> xyz=0.2808 -0.2225 0.01149 rpy=0 0 0
- joint front_right_wheel_joint: origin xyz=0 0 0 rpy=0 0 0 -> xyz=0.000739 -0.0743 -0.0373 rpy=0 0 0
- joint laser_joint: origin xyz=0.497 0 0.228 rpy=0 0 0 -> xyz=0.2503 -0.0018 0.1504 rpy=0 0 -3.14159
- joint rear_left_wheel_joint: origin xyz=0 0.295 0.12 rpy=0 0 0 -> xyz=-0.2458 0.29346 -0.027386 rpy=0 0 0
- joint rear_right_wheel_joint: origin xyz=0 -0.295 0.12 rpy=0 0 0 -> xyz=-0.2458 -0.2971 -0.027386 rpy=0 0 0

Commit message: fix: use original high-res R550 base mesh

File: r550_description/urdf/r550_ackermann.urdf (robot description, URDF)
Before this commit: robot r550_ackermann, 12 links, 11 joints
Links:
- link base_link: geometry collision box size=0.76 0.60 0.20; visual mesh filename=package://r550_description/reference/wheeltec_robot_urdf/me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

Commit message: fix: attach front wheels to R550 suspension knuckles

File: r550_description/urdf/r550_ackermann.urdf (robot description, URDF)
Before this commit: robot r550_ackermann, 12 links, 11 joints
Links:
- link front_left_steer_link: geometry collision box size=0.08 0.08 0.08; visual mesh filename=package://r550_description/meshes/r550_ackermann/front_left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
- link front_right_steer_link: geometry collision box size=0.08 0.08 0.08; visual mesh filename=package://r550_description/meshes/r550_ackermann/front_righ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
