Commit message: fix: remove dummy visible link from R550 model

File: r550_description/urdf/r550_ackermann_official.urdf (robot description, URDF)
Before this commit: robot top_akm_dl_robot, 13 links, 12 joints
Links:
- removed link steering_wheel_link
- link gyro_link: geometry 
Joints:
- removed joint steering_wheel_joint

Commit message: 使用复杂地图

File: r550_description/urdf/r550_ackermann_official.urdf (robot description, URDF)
Before this commit: robot top_akm_dl_robot, 12 links, 11 joints
Links:
- added link steering_wheel_link, mass 0.001
Joints:
- added joint steering_wheel_joint: type revolute, parent base_link, child steering_wheel_link, origin xyz=0.2 0 0.3 rpy=0 0 0, axis 0 0 1, limit lower=-0.52 upper=0.52 effort=1 velocity=1.0

Commit message: fix: lock front steering joints for planar drive

File: r550_description/urdf/r550_ackermann_official.urdf (robot description, URDF)
Before this commit: robot top_akm_dl_robot, 13 links, 12 joints
Joints:
- joint left1_joint: axis 0 0 1 -> (none); limit lower=-0.52 upper=0.52 effort=10 velocity=1.0 -> (none); type revolute -> fixed
- joint right1_joint: axis 0 0 1 -> (none); limit lower=-0.52 upper=0.52 effort=10 velocity=1.0 -> (none); type revolute -> fixed

Commit message: fix: 恢复 R550 前轮转向并改为后驱阿克曼控制
- 左/右前转向节由 fixed 改回 revolute，轴为 Z，限制 ±0.52 rad
- 四轮碰撞由高精度 STL 改为 0.1275 m 圆柱体，供 Gazebo 阿克曼插件计算轮半径
- 用 libgazebo_ros_ackermann_drive 替代 planar_move，实现后轮驱动+前轮转向
- 调低 PID 增益，避免小质量 R550 模型在 Gazebo ODE 下发散

File: r550_description/urdf/r550_ackermann_official.urdf (robot description, URDF)
Before this commit: robot top_akm_dl_robot, 13 links, 12 joints
Links:
- link lb_wheel_link: geometry collision cylinder length=0.08 radius=0.1275; visual mesh filename=package://r550_description/reference/wheeltec_robot_urdf/me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
- link lf_wheel_link: geometry collision cylinder length=0.08 radius=0.1275; visual mesh filename=package://r550_description/reference/wheeltec_robot_urdf/me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
- link rb_wheel_link: geometry collision cylinder length=0.08 radius=0.1275; visual mesh filename=package://r550_description/reference/wheeltec_robot_urdf/me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
- link rf_wheel_link: geometry collision cylinder length=0.08 radius=0.1275; visual mesh filename=package://r550_description/reference/wheeltec_robot_urdf/me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
Joints:
- joint left1_joint: axis (none) -> 0 0 1; limit (none) -> lower=-0.52 upper=0.52 effort=20 velocity=2.0; type fixed -> revolute
- joint right1_joint: axis (none) -> 0 0 1; limit (none) -> lower=-0.52 upper=0.52 effort=20 velocity=2.0; type fixed -> revolute

Commit message: fix: 稳定 R550 倒车与碰撞响应
- 线性速度 PID 去掉微分项，避免 0.3~0.4 m/s 倒车时数值发散
- 车体碰撞由高精度 STL 换成简化盒，摄像头/激光/控制器仅保留视觉，降低撞柱爆炸风险
- 增加轮胎接触刚度/阻尼参数，限制最大仿真速度 0.4 m/s
- 出生点移到南侧长走廊，前后预留足够直线/倒车空间
- 新增 scripts/test_sim_motion.sh 自动回归前进、倒车、快速倒车和左转

File: r550_description/urdf/r550_ackermann_official.urdf (robot description, URDF)
Before this commit: robot top_akm_dl_robot, 13 links, 12 joints
Links:
- link base_link: geometry collision box size=0.762 0.632 0.228; visual mesh filename=package://r550_description/reference/wheeltec_robot_urdf/me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
- link camera_link: geometry visual mesh filename=package://r550_description/reference/wheeltec_robot_urdf/me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
- link controller_link: geometry visual mesh filename=package://r550_description/reference/wheeltec_robot_urdf/me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
- link laser_link: geometry visual mesh filename=package://r550_description/reference/wheeltec_robot_urdf/me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
